File: ath-dbg.kicad_pcb (KiCad board)
At the start: 4 copper layers, 89.6 x 63.2 mm, 47 parts, among them J1 TWL_WifiConn_Rcpt, J10 CortexDbgConn SMD, J2 Conn_01x08, J3 CortexDbgConn, J4 Conn_01x05, J5 Conn_01x08, J6 Conn_01x04, U1 Pico, U2 TLV70018DDC, U3 TXU0304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

Commit message: reset stuff
Parts:
- added R19: 47k, Resistor_SMD:R_0603_1608Metric_Pad0.98x0.95mm_HandSolder, F.Cu at (130.0, 87.8)
- J2: value Conn_01x08 -> Conn_01x09; footprint Connector_PinHeader_2.54mm:PinHeader_1x08_P2.54mm_Vertical -> Connector_PinHeader_2.54mm:PinHeader_1x09_P2.54mm_Vertical
- J4: footprint Connector_PinHeader_2.54mm:PinHeader_1x05_P2.54mm_Vertical -> Connector_PinHeader_2.54mm:PinHeader_1x06_P2.54mm_Vertical
- moved REF** 4.51 mm to (170.5, 90.7)
Connections:
- J10 pad 10: JTAG33.ERST -> JTAG33.CPURST
- J3 pad 10: JTAG33.ERST -> JTAG33.CPURST
- J4 pad 4: +1V8 -> JTAG18.CPURST
- J4 pad 5: GND -> +1V8
- U1 pad 34: unconnected-(U1-GPIO28_ADC2-Pad34) -> JTAG33.CPURST
- U5 pad 11: unconnected-(U5-B3Y-Pad11) -> JTAG18.CPURST
- U5 pad 4: unconnected-(U5-A3-Pad4) -> JTAG33.CPURST
Routing:
- net JTAG33.CPURST: track 0.00 -> 126.1 mm, vias 0 -> 1
- net JTAG33.ERST: track 94.5 -> 57.6 mm
- net JTAG18.CPURST: track 0.00 -> 32.5 mm, vias 0 -> 1
- net +1V8: track 117.3 -> 122.2 mm
- net +3V3: track 256.6 -> 259.3 mm, vias 7 -> 8
- net GND: vias 21 -> 27
Other:
- board text added: "Pico pinout: * GP00: UART RP to Ath/DWM (R2A) * GP01: UART Ath/DWM to RP (A2R) * GP02: JTAG.ERST (debug CPU reset extension) * GP03: JTAG.TRST * GP04: ~{WIFI_RST} (Ath chip reset) * GP05: SPI.~{WP} * GP06: nSEL_ATH (0=Ath/DWM/TWL, 1=NTR wifi) * GP07: 32 kHz clock to DWM * GP08: SPI.CIPO * GP09: SPI.~{CS} * GP10: SPI.SCK * GP11: SPI.COPI * GP12: JTAG.TDO * GP13: JTAG.TCK * GP14: JTAG.TDI * GP15: J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"
- board text added: "nRST"
- board text removed: "Pico pinout: * GP00: UART RP to Ath/DWM (R2A) * GP01: UART Ath/DWM to RP (A2R) * GP02: JTAG.ERST (debug CPU reset extension) * GP03: JTAG.TRST * GP04: ~{WIFI_RST} * GP05: SPI.~{WP} * GP06: nSEL_ATH (0=Ath/DWM/TWL, 1=NTR wifi) * GP07: 32 kHz clock to DWM * GP08: SPI.CIPO * GP09: SPI.~{CS} * GP10: SPI.SCK * GP11: SPI.COPI * GP12: JTAG.TDO * GP13: JTAG.TCK * GP14: JTAG.TDI * GP15: JTAG.TMS * GP16: S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"
