File: ath-dbg.kicad_sch (KiCad schematic)
At the start: 55 parts, among them J1 TWL_WifiConn_Rcpt, J10 CortexDbgConn SMD, J11 TWL_UART_A2R, J12 TWL_UART_R2A, J2 Conn_01x08, J3 CortexDbgConn, J4 Conn_01x05, J5 Conn_01x08, J6 Conn_01x04, J7 EJTAG_RST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

Commit message: reset stuff
Parts:
- added R19: 47k, Resistor_SMD:R_0603_1608Metric_Pad0.98x0.95mm_HandSolder, symbol Device:R_Small_US
- J2: value Conn_01x08 -> Conn_01x09; footprint Connector_PinHeader_2.54mm:PinHeader_1x08_P2.54mm_Vertical -> Connector_PinHeader_2.54mm:PinHeader_1x09_P2.54mm_Vertical; symbol Connector_Generic:Conn_01x08 -> Connector_Generic:Conn_01x09
- J4: footprint Connector_PinHeader_2.54mm:PinHeader_1x05_P2.54mm_Vertical -> Connector_PinHeader_2.54mm:PinHeader_1x06_P2.54mm_Vertical; symbol Connector_Generic:Conn_01x05 -> Connector_Generic:Conn_01x06
- renumbered R19 to R20
Connections:
- net +1V8: now also J4.5 (Pin_5); no longer J4.4 (Pin_4)
- net +3V3: now also R19.1
- net GND: now also J4.6 (Pin_6); no longer J4.5 (Pin_5)
- net JTAG33.ERST: no longer J10.10 (Pin_10), J3.10 (Pin_10)
- net JTAG18.CPURST: now reaches U5.11 (B3Y)
- net JTAG18.CPURST: now also J4.4 (Pin_4)
- net JTAG33.CPURST: now reaches U5.4 (A3)
- net JTAG33.CPURST: now also J10.10 (Pin_10), J2.9 (Pin_9), J3.10 (Pin_10), U1.34 (GPIO28_ADC2), R19.2
- no-connect marks 29 -> 25
Other:
- moved on the sheet: R13, R14, R15
